Commit message: Test hospital world

File: src/yahboom_M3Pro_description/urdf/M3Pro.urdf (robot description, URDF)
Before this commit: robot M3Pro, 20 links, 19 joints
Links:
- added link base_footprint
- link arm_base_Link: geometry visual mesh filename=package://yahboom_M3Pro_description/meshes/arm_base_Link.STL
- link base_link: geometry collision box size=0.2 0.16 0.06; visual mesh filename=package://yahboom_M3Pro_description/meshes/base_link.STL
- link lwheel1: geometry collision cylinder length=0.02 radius=0.04; visual cylinder length=0.02 radius=0.04
- link lwheel2: geometry collision cylinder length=0.02 radius=0.04; visual cylinder length=0.02 radius=0.04
- link rwheel1: geometry collision cylinder length=0.02 radius=0.04; visual cylinder length=0.02 radius=0.04
- link rwheel2: geometry collision cylinder length=0.02 radius=0.04; visual cylinder length=0.02 radius=0.04
Joints:
- added joint base_joint: type fixed, parent base_footprint, child base_link, origin xyz=0 0 0.04 rpy=0 0 0
- joint lwheel1_Joint: limit lower=0 upper=0 effort=0 velocity=0 -> (none); type revolute -> continuous
- joint lwheel2_Joint: limit lower=0 upper=0 effort=0 velocity=0 -> (none); type revolute -> continuous
- joint rwheel1_Joint: limit lower=0 upper=0 effort=0 velocity=0 -> (none); type revolute -> continuous
- joint rwheel2_Joint: limit lower=0 upper=0 effort=0 velocity=0 -> (none); type revolute -> continuous

Commit message: Update urdf

File: src/yahboom_M3Pro_description/urdf/M3Pro.urdf (robot description, URDF)
Before this commit: robot M3Pro, 21 links, 20 joints
Links:
- link lwheel1: geometry collision cylinder length=0.02 radius=0.04; visual mesh filename=package://yahboom_M3Pro_description/meshes/lwheel1.STL
- link lwheel2: geometry collision cylinder length=0.02 radius=0.04; visual mesh filename=package://yahboom_M3Pro_description/meshes/lwheel2.STL
- link rwheel1: geometry collision cylinder length=0.02 radius=0.04; visual mesh filename=package://yahboom_M3Pro_description/meshes/rwheel1.STL
- link rwheel2: geometry collision cylinder length=0.02 radius=0.04; visual mesh filename=package://yahboom_M3Pro_description/meshes/rwheel2.STL
Joints:
- removed joint arm4_Joiint
- added joint arm4_Joint: type fixed, parent arm3, child arm4, origin xyz=0 0 0.08285 rpy=0 0.785 -0.027075, axis -2.6392E-05 -1 0, limit lower=-1.5708 upper=1.5708 effort=100 velocity=1
- joint arm1_Joint: type revolute -> fixed
- joint arm2_Joint: type revolute -> fixed
- joint arm3_Joint: origin xyz=0 0 0.08285 rpy=6.3702E-05 0 0.027102 -> xyz=0 0 0.08285 rpy=6.3702E-05 0.785 0.027102; type revolute -> fixed
- joint arm5_Joint: type revolute -> fixed
- joint llink1_Joint: type continuous -> fixed
- joint llink2_Joint: type continuous -> fixed
- joint llink3_Joint: type continuous -> fixed
- joint rlink1_Joint: type revolute -> fixed
- joint rlink2_Joint: type continuous -> fixed
- joint rlink3_Joint: type continuous -> fixed

Commit message: Enabled DepthCam on M3Pro in Gazebo and Rviz

File: src/yahboom_M3Pro_description/urdf/M3Pro.urdf (robot description, URDF)
Before this commit: robot M3Pro, 21 links, 20 joints
Links:
- added link camera_optical_link
Joints:
- added joint camera_optical_joint: type fixed, parent DCW2, child camera_optical_link, origin xyz=0 0 0 rpy=${-pi/2} 0 ${-pi/2}
- joint arm4_Joint: origin xyz=0 0 0.08285 rpy=0 0.785 -0.027075 -> xyz=0 0 0.08285 rpy=0 ${pi/4.7} -0.027075

Commit message: Add all-in-one launcn

File: src/yahboom_M3Pro_description/urdf/M3Pro.urdf (robot description, URDF)
Before this commit: robot M3Pro, 22 links, 21 joints
Links:
- link base_link: mass 0.870994544286568 -> 2
Joints:
- joint Camera_Joint: type revolute -> fixed
- joint arm2_Joint: origin xyz=-0.0021522 6.1185E-05 0.033 rpy=-6.3725E-05 0 -0.028422 -> xyz=-0.0021522 6.1185E-05 0.033 rpy=-6.3725E-05 -${pi/4} -0.028422
- joint arm3_Joint: origin xyz=0 0 0.08285 rpy=6.3702E-05 0.785 0.027102 -> xyz=0 0 0.08285 rpy=6.3702E-05 ${pi/2} 0.027102
- joint rwheel1_Joint: axis 0 0 -1 -> 0 0 1
- joint rwheel2_Joint: axis 0 0 -1 -> 0 0 1

Commit message: Add slam_toolbox trial

File: src/yahboom_M3Pro_description/urdf/M3Pro.urdf (robot description, URDF)
Before this commit: robot M3Pro, 22 links, 21 joints
Joints:
- joint arm4_Joint: origin xyz=0 0 0.08285 rpy=0 ${pi/4.7} -0.027075 -> xyz=0 0 0.08285 rpy=0 ${pi/4.8} -0.027075

Commit message: Update hospital world

File: src/yahboom_M3Pro_description/urdf/M3Pro.urdf (robot description, URDF)
Before this commit: robot M3Pro, 22 links, 21 joints
Links:
- link base_link: mass 2 -> 4
Joints:
- joint arm1_Joint: origin xyz=0.033617 -1.2421E-05 0.185 rpy=6.3751E-05 0 0.028395 -> xyz=0.033617 -1.2421E-05 0.185 rpy=0 0 0
- joint arm2_Joint: origin xyz=-0.0021522 6.1185E-05 0.033 rpy=-6.3725E-05 -${pi/4} -0.028422 -> xyz=-0.0021522 6.1185E-05 0.033 rpy=0 -${pi/4} 0
- joint arm3_Joint: origin xyz=0 0 0.08285 rpy=6.3702E-05 ${pi/2} 0.027102 -> xyz=0 0 0.08285 rpy=0 ${pi/2} 0
- joint arm4_Joint: origin xyz=0 0 0.08285 rpy=0 ${pi/4.8} -0.027075 -> xyz=0 0 0.08285 rpy=0 ${pi/4} 0

Commit message: Two LiDAR SLAM

File: src/yahboom_M3Pro_description/urdf/M3Pro.urdf (robot description, URDF)
Before this commit: robot M3Pro, 22 links, 21 joints
Links:
- added link laser_front_right_link; visual cylinder length=0.03 radius=0.02
- added link laser_rear_left_link; visual cylinder length=0.03 radius=0.02
Joints:
- added joint laser_front_right_joint: type fixed, parent base_link, child laser_front_right_link, origin xyz=0.12 -0.10 0.08 rpy=0 0 0
- added joint laser_rear_left_joint: type fixed, parent base_link, child laser_rear_left_link, origin xyz=-0.12 0.10 0.08 rpy=0 0 ${pi}

Commit message: Use ROS2 controller

File: src/yahboom_M3Pro_description/urdf/M3Pro.urdf (robot description, URDF)
Before this commit: robot M3Pro, 24 links, 23 joints
Links:
- link base_link: mass 4 -> 4.0
Joints:
- joint lwheel1_Joint: limit (none) -> effort=10.0 velocity=20.0
- joint lwheel2_Joint: limit (none) -> effort=10.0 velocity=20.0
- joint rwheel1_Joint: limit (none) -> effort=10.0 velocity=20.0
- joint rwheel2_Joint: limit (none) -> effort=10.0 velocity=20.0
