Commit message: Build C++ node to merge multi-lidar scan data

File: src/yahboom_m3pro_slam_demo/urdf/.ipynb_checkpoints/M3Pro-checkpoint.urdf (robot description, URDF)
Before this commit: robot M3Pro, 24 links, 23 joints
Links:
- removed link base_footprint
- removed link camera_optical_link
- removed link laser_front_right_link
- removed link laser_rear_left_link
- link Camera: geometry collision mesh filename=package://yahboom_m3pro_slam_demo/meshes/Camera.STL; visual mesh filename=package://yahboom_m3pro_slam_demo/meshes/Camera.STL
- link DCW2: geometry collision mesh filename=package://yahboom_m3pro_slam_demo/meshes/DCW2.STL; visual mesh filename=package://yahboom_m3pro_slam_demo/meshes/DCW2.STL
- link Gripping: geometry collision mesh filename=package://yahboom_m3pro_slam_demo/meshes/Gripping.STL; visual mesh filename=package://yahboom_m3pro_slam_demo/meshes/Gripping.STL
- link arm1: geometry collision mesh filename=package://yahboom_m3pro_slam_demo/meshes/arm1.STL; visual mesh filename=package://yahboom_m3pro_slam_demo/meshes/arm1.STL
- link arm2: geometry collision mesh filename=package://yahboom_m3pro_slam_demo/meshes/arm2.STL; visual mesh filename=package://yahboom_m3pro_slam_demo/meshes/arm2.STL
- link arm3: geometry collision mesh filename=package://yahboom_m3pro_slam_demo/meshes/arm3.STL; visual mesh filename=package://yahboom_m3pro_slam_demo/meshes/arm3.STL
- link arm4: geometry collision mesh filename=package://yahboom_m3pro_slam_demo/meshes/arm4.STL; visual mesh filename=package://yahboom_m3pro_slam_demo/meshes/arm4.STL
- link arm5: geometry collision mesh filename=package://yahboom_m3pro_slam_demo/meshes/arm5.STL; visual mesh filename=package://yahboom_m3pro_slam_demo/meshes/arm5.STL
- link arm_base_Link: geometry collision mesh filename=package://yahboom_m3pro_slam_demo/meshes/arm_base_Link.STL; visual mesh filename=package://yahboom_m3pro_slam_demo/meshes/arm_base_Link.STL
- link base_link: mass 4.0 -> 0.870994544286568; geometry collision mesh filename=package://yahboom_m3pro_slam_demo/meshes/base_link.STL; visual mesh filename=package://yahboom_m3pro_slam_demo/meshes/base_link.STL
- link llink1: geometry collision mesh filename=package://yahboom_m3pro_slam_demo/meshes/llink1.STL; visual mesh filename=package://yahboom_m3pro_slam_demo/meshes/llink1.STL
- link llink2: geometry collision mesh filename=package://yahboom_m3pro_slam_demo/meshes/llink2.STL; visual mesh filename=package://yahboom_m3pro_slam_demo/meshes/llink2.STL
- link llink3: geometry collision mesh filename=package://yahboom_m3pro_slam_demo/meshes/llink3.STL; visual mesh filename=package://yahboom_m3pro_slam_demo/meshes/llink3.STL
- link lwheel1: geometry collision mesh filename=package://yahboom_m3pro_slam_demo/meshes/lwheel1.STL; visual mesh filename=package://yahboom_m3pro_slam_demo/meshes/lwheel1.STL
- link lwheel2: geometry collision mesh filename=package://yahboom_m3pro_slam_demo/meshes/lwheel2.STL; visual mesh filename=package://yahboom_m3pro_slam_demo/meshes/lwheel2.STL
- link rlink1: geometry collision mesh filename=package://yahboom_m3pro_slam_demo/meshes/rlink1.STL; visual mesh filename=package://yahboom_m3pro_slam_demo/meshes/rlink1.STL
- link rlink2: geometry collision mesh filename=package://yahboom_m3pro_slam_demo/meshes/rlink2.STL; visual mesh filename=package://yahboom_m3pro_slam_demo/meshes/rlink2.STL
- link rlink3: geometry collision mesh filename=package://yahboom_m3pro_slam_demo/meshes/rlink3.STL; visual mesh filename=package://yahboom_m3pro_slam_demo/meshes/rlink3.STL
- link rwheel1: geometry collision mesh filename=package://yahboom_m3pro_slam_demo/meshes/rwheel1.STL; visual mesh filename=package://yahboom_m3pro_slam_demo/meshes/rwheel1.STL
- link rwheel2: geometry collision mesh filename=package://yahboom_m3pro_slam_demo/meshes/rwheel2.STL; visual mesh filename=package://yahboom_m3pro_slam_demo/meshes/rwheel2.STL
Joints:
- removed joint arm4_Joint
- removed joint base_joint
- removed joint camera_optical_joint
- removed joint laser_front_right_joint
- removed joint laser_rear_left_joint
- added joint arm4_Joiint: type revolute, parent arm3, child arm4, origin xyz=0 0 0.08285 rpy=0 0 -0.027075, axis -2.6392E-05 -1 0, limit lower=-1.5708 upper=1.5708 effort=100 velocity=1
- joint Camera_Joint: type fixed -> revolute
- joint arm1_Joint: origin xyz=0.033617 -1.2421E-05 0.185 rpy=0 0 0 -> xyz=0.033617 -1.2421E-05 0.185 rpy=6.3751E-05 0 0.028395; type fixed -> revolute
- joint arm2_Joint: origin xyz=-0.0021522 6.1185E-05 0.033 rpy=0 -${pi/4} 0 -> xyz=-0.0021522 6.1185E-05 0.033 rpy=-6.3725E-05 0 -0.028422; type fixed -> revolute
- joint arm3_Joint: origin xyz=0 0 0.08285 rpy=0 ${pi/2} 0 -> xyz=0 0 0.08285 rpy=6.3702E-05 0 0.027102; type fixed -> revolute
- joint arm5_Joint: type fixed -> revolute
- joint llink1_Joint: type fixed -> continuous
- joint llink2_Joint: type fixed -> continuous
- joint llink3_Joint: type fixed -> continuous
- joint lwheel1_Joint: limit effort=10.0 velocity=20.0 -> lower=0 upper=0 effort=0 velocity=0; type continuous -> revolute
- joint lwheel2_Joint: limit effort=10.0 velocity=20.0 -> lower=0 upper=0 effort=0 velocity=0; type continuous -> revolute
- joint rlink1_Joint: type fixed -> revolute
- joint rlink2_Joint: type fixed -> continuous
- joint rlink3_Joint: type fixed -> continuous
- joint rwheel1_Joint: axis 0 0 1 -> 0 0 -1; limit effort=10.0 velocity=20.0 -> lower=0 upper=0 effort=0 velocity=0; type continuous -> revolute
- joint rwheel2_Joint: axis 0 0 1 -> 0 0 -1; limit effort=10.0 velocity=20.0 -> lower=0 upper=0 effort=0 velocity=0; type continuous -> revolute

File: src/yahboom_m3pro_slam_demo/urdf/M3Pro.urdf (robot description, URDF)
Before this commit: robot M3Pro, 20 links, 19 joints
Links:
- added link base_footprint
- added link camera_optical_link
- added link laser_front_right_link; visual cylinder length=0.03 radius=0.02
- added link laser_rear_left_link; visual cylinder length=0.03 radius=0.02
- link Camera: geometry collision mesh filename=package://yahboom_m3pro_slam_demo/meshes/Camera.STL; visual mesh filename=package://yahboom_m3pro_slam_demo/meshes/Camera.STL
- link DCW2: geometry collision mesh filename=package://yahboom_m3pro_slam_demo/meshes/DCW2.STL; visual mesh filename=package://yahboom_m3pro_slam_demo/meshes/DCW2.STL
- link Gripping: geometry collision mesh filename=package://yahboom_m3pro_slam_demo/meshes/Gripping.STL; visual mesh filename=package://yahboom_m3pro_slam_demo/meshes/Gripping.STL
- link arm1: geometry collision mesh filename=package://yahboom_m3pro_slam_demo/meshes/arm1.STL; visual mesh filename=package://yahboom_m3pro_slam_demo/meshes/arm1.STL
- link arm2: geometry collision mesh filename=package://yahboom_m3pro_slam_demo/meshes/arm2.STL; visual mesh filename=package://yahboom_m3pro_slam_demo/meshes/arm2.STL
- link arm3: geometry collision mesh filename=package://yahboom_m3pro_slam_demo/meshes/arm3.STL; visual mesh filename=package://yahboom_m3pro_slam_demo/meshes/arm3.STL
- link arm4: geometry collision mesh filename=package://yahboom_m3pro_slam_demo/meshes/arm4.STL; visual mesh filename=package://yahboom_m3pro_slam_demo/meshes/arm4.STL
- link arm5: geometry collision mesh filename=package://yahboom_m3pro_slam_demo/meshes/arm5.STL; visual mesh filename=package://yahboom_m3pro_slam_demo/meshes/arm5.STL
- link arm_base_Link: geometry visual mesh filename=package://yahboom_m3pro_slam_demo/meshes/arm_base_Link.STL
- link base_link: mass 0.870994544286568 -> 4.0; geometry collision box size=0.2 0.16 0.06; visual mesh filename=package://yahboom_m3pro_slam_demo/meshes/base_link.STL
- link llink1: geometry collision mesh filename=package://yahboom_m3pro_slam_demo/meshes/llink1.STL; visual mesh filename=package://yahboom_m3pro_slam_demo/meshes/llink1.STL
- link llink2: geometry collision mesh filename=package://yahboom_m3pro_slam_demo/meshes/llink2.STL; visual mesh filename=package://yahboom_m3pro_slam_demo/meshes/llink2.STL
- link llink3: geometry collision mesh filename=package://yahboom_m3pro_slam_demo/meshes/llink3.STL; visual mesh filename=package://yahboom_m3pro_slam_demo/meshes/llink3.STL
- link lwheel1: geometry collision cylinder length=0.02 radius=0.04; visual mesh filename=package://yahboom_m3pro_slam_demo/meshes/lwheel1.STL
- link lwheel2: geometry collision cylinder length=0.02 radius=0.04; visual mesh filename=package://yahboom_m3pro_slam_demo/meshes/lwheel2.STL
- link rlink1: geometry collision mesh filename=package://yahboom_m3pro_slam_demo/meshes/rlink1.STL; visual mesh filename=package://yahboom_m3pro_slam_demo/meshes/rlink1.STL
- link rlink2: geometry collision mesh filename=package://yahboom_m3pro_slam_demo/meshes/rlink2.STL; visual mesh filename=package://yahboom_m3pro_slam_demo/meshes/rlink2.STL
- link rlink3: geometry collision mesh filename=package://yahboom_m3pro_slam_demo/meshes/rlink3.STL; visual mesh filename=package://yahboom_m3pro_slam_demo/meshes/rlink3.STL
- link rwheel1: geometry collision cylinder length=0.02 radius=0.04; visual mesh filename=package://yahboom_m3pro_slam_demo/meshes/rwheel1.STL
- link rwheel2: geometry collision cylinder length=0.02 radius=0.04; visual mesh filename=package://yahboom_m3pro_slam_demo/meshes/rwheel2.STL
Joints:
- removed joint arm4_Joiint
- added joint arm4_Joint: type fixed, parent arm3, child arm4, origin xyz=0 0 0.08285 rpy=0 ${pi/4} 0, axis -2.6392E-05 -1 0, limit lower=-1.5708 upper=1.5708 effort=100 velocity=1
- added joint base_joint: type fixed, parent base_footprint, child base_link, origin xyz=0 0 0.04 rpy=0 0 0
- added joint camera_optical_joint: type fixed, parent DCW2, child camera_optical_link, origin xyz=0 0 0 rpy=${-pi/2} 0 ${-pi/2}
- added joint laser_front_right_joint: type fixed, parent base_link, child laser_front_right_link, origin xyz=0.12 -0.10 0.08 rpy=0 0 0
- added joint laser_rear_left_joint: type fixed, parent base_link, child laser_rear_left_link, origin xyz=-0.12 0.10 0.08 rpy=0 0 ${pi}
- joint Camera_Joint: type revolute -> fixed
- joint arm1_Joint: origin xyz=0.033617 -1.2421E-05 0.185 rpy=6.3751E-05 0 0.028395 -> xyz=0.033617 -1.2421E-05 0.185 rpy=0 0 0; type revolute -> fixed
- joint arm2_Joint: origin xyz=-0.0021522 6.1185E-05 0.033 rpy=-6.3725E-05 0 -0.028422 -> xyz=-0.0021522 6.1185E-05 0.033 rpy=0 -${pi/4} 0; type revolute -> fixed
- joint arm3_Joint: origin xyz=0 0 0.08285 rpy=6.3702E-05 0 0.027102 -> xyz=0 0 0.08285 rpy=0 ${pi/2} 0; type revolute -> fixed
- joint arm5_Joint: type revolute -> fixed
- joint llink1_Joint: type continuous -> fixed
- joint llink2_Joint: type continuous -> fixed
- joint llink3_Joint: type continuous -> fixed
- joint lwheel1_Joint: limit lower=0 upper=0 effort=0 velocity=0 -> effort=10.0 velocity=20.0; type revolute -> continuous
- joint lwheel2_Joint: limit lower=0 upper=0 effort=0 velocity=0 -> effort=10.0 velocity=20.0; type revolute -> continuous
- joint rlink1_Joint: type revolute -> fixed
- joint rlink2_Joint: type continuous -> fixed
- joint rlink3_Joint: type continuous -> fixed
- joint rwheel1_Joint: axis 0 0 -1 -> 0 0 1; limit lower=0 upper=0 effort=0 velocity=0 -> effort=10.0 velocity=20.0; type revolute -> continuous
- joint rwheel2_Joint: axis 0 0 -1 -> 0 0 1; limit lower=0 upper=0 effort=0 velocity=0 -> effort=10.0 velocity=20.0; type revolute -> continuous
