Commit message: Updated urdf for lidar positions

File: src/yahboom_m3pro_slam_demo/urdf/M3Pro.urdf (robot description, URDF)
Before this commit: robot M3Pro, 24 links, 23 joints
Links:
- added link laser_front_right; visual cylinder length=0.03 radius=0.019
- added link laser_rear_left; visual cylinder length=0.03 radius=0.019
Joints:
- added joint laser_front_right_Joint: type fixed, parent base_link, child laser_front_right, origin xyz=0.10386 -0.09160 0.1253 rpy=0 0 0, axis 0 0 0, limit lower=0 upper=0 effort=0 velocity=0
- added joint laser_rear_left_Joint: type fixed, parent base_link, child laser_rear_left, origin xyz=-0.11867 0.09 0.1253 rpy=0 0 0, axis 0 0 0, limit lower=0 upper=0 effort=0 velocity=0

Commit message: calcuate LiDAR position directly from urdf

File: src/yahboom_m3pro_slam_demo/urdf/M3Pro.urdf (robot description, URDF)
Before this commit: robot M3Pro, 26 links, 25 joints
Links:
- removed link laser_front_right
- removed link laser_rear_left
- added link laser_front; visual cylinder length=0.03 radius=0.019
- added link laser_rear; visual cylinder length=0.03 radius=0.019
Joints:
- removed joint laser_front_right_Joint
- removed joint laser_front_right_joint
- removed joint laser_rear_left_Joint
- removed joint laser_rear_left_joint
- added joint laser_front_joint: type fixed, parent base_link, child laser_front, origin xyz=0.10386 -0.09160 0.1253 rpy=0 0 0, axis 0 0 0, limit lower=0 upper=0 effort=0 velocity=0
- added joint laser_front_right_joint_to_remove: type fixed, parent base_link, child laser_front_right_link, origin xyz=0.12 -0.10 0.08 rpy=0 0 0
- added joint laser_rear_joint: type fixed, parent base_link, child laser_rear, origin xyz=-0.11867 0.09 0.1253 rpy=0 0 ${pi}, axis 0 0 0, limit lower=0 upper=0 effort=0 velocity=0
- added joint laser_rear_left_joint_to_remove: type fixed, parent base_link, child laser_rear_left_link, origin xyz=-0.12 0.10 0.08 rpy=0 0 ${pi}
