Commit message: Refactor and add IMU&EKF for SLAM

File: src/m3pro_world_bringup/urdf/.ipynb_checkpoints/M3Pro-checkpoint.urdf (robot description, URDF)
Before this commit: robot M3Pro, 20 links, 19 joints
Links:
- link Camera: geometry collision mesh filename=package://m3pro_world_bringup/meshes/Camera.STL; visual mesh filename=package://m3pro_world_bringup/meshes/Camera.STL
- link DCW2: geometry collision mesh filename=package://m3pro_world_bringup/meshes/DCW2.STL; visual mesh filename=package://m3pro_world_bringup/meshes/DCW2.STL
- link Gripping: geometry collision mesh filename=package://m3pro_world_bringup/meshes/Gripping.STL; visual mesh filename=package://m3pro_world_bringup/meshes/Gripping.STL
- link arm1: geometry collision mesh filename=package://m3pro_world_bringup/meshes/arm1.STL; visual mesh filename=package://m3pro_world_bringup/meshes/arm1.STL
- link arm2: geometry collision mesh filename=package://m3pro_world_bringup/meshes/arm2.STL; visual mesh filename=package://m3pro_world_bringup/meshes/arm2.STL
- link arm3: geometry collision mesh filename=package://m3pro_world_bringup/meshes/arm3.STL; visual mesh filename=package://m3pro_world_bringup/meshes/arm3.STL
- link arm4: geometry collision mesh filename=package://m3pro_world_bringup/meshes/arm4.STL; visual mesh filename=package://m3pro_world_bringup/meshes/arm4.STL
- link arm5: geometry collision mesh filename=package://m3pro_world_bringup/meshes/arm5.STL; visual mesh filename=package://m3pro_world_bringup/meshes/arm5.STL
- link arm_base_Link: geometry collision mesh filename=package://m3pro_world_bringup/meshes/arm_base_Link.STL; visual mesh filename=package://m3pro_world_bringup/meshes/arm_base_Link.STL
- link base_link: geometry collision mesh filename=package://m3pro_world_bringup/meshes/base_link.STL; visual mesh filename=package://m3pro_world_bringup/meshes/base_link.STL
- link llink1: geometry collision mesh filename=package://m3pro_world_bringup/meshes/llink1.STL; visual mesh filename=package://m3pro_world_bringup/meshes/llink1.STL
- link llink2: geometry collision mesh filename=package://m3pro_world_bringup/meshes/llink2.STL; visual mesh filename=package://m3pro_world_bringup/meshes/llink2.STL
- link llink3: geometry collision mesh filename=package://m3pro_world_bringup/meshes/llink3.STL; visual mesh filename=package://m3pro_world_bringup/meshes/llink3.STL
- link lwheel1: geometry collision mesh filename=package://m3pro_world_bringup/meshes/lwheel1.STL; visual mesh filename=package://m3pro_world_bringup/meshes/lwheel1.STL
- link lwheel2: geometry collision mesh filename=package://m3pro_world_bringup/meshes/lwheel2.STL; visual mesh filename=package://m3pro_world_bringup/meshes/lwheel2.STL
- link rlink1: geometry collision mesh filename=package://m3pro_world_bringup/meshes/rlink1.STL; visual mesh filename=package://m3pro_world_bringup/meshes/rlink1.STL
- link rlink2: geometry collision mesh filename=package://m3pro_world_bringup/meshes/rlink2.STL; visual mesh filename=package://m3pro_world_bringup/meshes/rlink2.STL
- link rlink3: geometry collision mesh filename=package://m3pro_world_bringup/meshes/rlink3.STL; visual mesh filename=package://m3pro_world_bringup/meshes/rlink3.STL
- link rwheel1: geometry collision mesh filename=package://m3pro_world_bringup/meshes/rwheel1.STL; visual mesh filename=package://m3pro_world_bringup/meshes/rwheel1.STL
- link rwheel2: geometry collision mesh filename=package://m3pro_world_bringup/meshes/rwheel2.STL; visual mesh filename=package://m3pro_world_bringup/meshes/rwheel2.STL

File: src/m3pro_world_bringup/urdf/M3Pro.urdf (robot description, URDF)
Before this commit: robot M3Pro, 26 links, 25 joints
Links:
- removed link laser_front_right_link
- removed link laser_rear_left_link
- link Camera: geometry collision mesh filename=package://m3pro_world_bringup/meshes/Camera.STL; visual mesh filename=package://m3pro_world_bringup/meshes/Camera.STL
- link DCW2: geometry collision mesh filename=package://m3pro_world_bringup/meshes/DCW2.STL; visual mesh filename=package://m3pro_world_bringup/meshes/DCW2.STL
- link Gripping: geometry collision mesh filename=package://m3pro_world_bringup/meshes/Gripping.STL; visual mesh filename=package://m3pro_world_bringup/meshes/Gripping.STL
- link arm1: geometry collision mesh filename=package://m3pro_world_bringup/meshes/arm1.STL; visual mesh filename=package://m3pro_world_bringup/meshes/arm1.STL
- link arm2: geometry collision mesh filename=package://m3pro_world_bringup/meshes/arm2.STL; visual mesh filename=package://m3pro_world_bringup/meshes/arm2.STL
- link arm3: geometry collision mesh filename=package://m3pro_world_bringup/meshes/arm3.STL; visual mesh filename=package://m3pro_world_bringup/meshes/arm3.STL
- link arm4: geometry collision mesh filename=package://m3pro_world_bringup/meshes/arm4.STL; visual mesh filename=package://m3pro_world_bringup/meshes/arm4.STL
- link arm5: geometry collision mesh filename=package://m3pro_world_bringup/meshes/arm5.STL; visual mesh filename=package://m3pro_world_bringup/meshes/arm5.STL
- link arm_base_Link: geometry visual mesh filename=package://m3pro_world_bringup/meshes/arm_base_Link.STL
- link base_link: geometry collision box size=0.2 0.16 0.06; visual mesh filename=package://m3pro_world_bringup/meshes/base_link.STL
- link laser_front: geometry collision cylinder length=0.03 radius=0.019; visual cylinder length=0.03 radius=0.019
- link laser_rear: geometry collision cylinder length=0.03 radius=0.019; visual cylinder length=0.03 radius=0.019
- link llink1: geometry collision mesh filename=package://m3pro_world_bringup/meshes/llink1.STL; visual mesh filename=package://m3pro_world_bringup/meshes/llink1.STL
- link llink2: geometry collision mesh filename=package://m3pro_world_bringup/meshes/llink2.STL; visual mesh filename=package://m3pro_world_bringup/meshes/llink2.STL
- link llink3: geometry collision mesh filename=package://m3pro_world_bringup/meshes/llink3.STL; visual mesh filename=package://m3pro_world_bringup/meshes/llink3.STL
- link lwheel1: geometry collision cylinder length=0.02 radius=0.04; visual mesh filename=package://m3pro_world_bringup/meshes/lwheel1.STL
- link lwheel2: geometry collision cylinder length=0.02 radius=0.04; visual mesh filename=package://m3pro_world_bringup/meshes/lwheel2.STL
- link rlink1: geometry collision mesh filename=package://m3pro_world_bringup/meshes/rlink1.STL; visual mesh filename=package://m3pro_world_bringup/meshes/rlink1.STL
- link rlink2: geometry collision mesh filename=package://m3pro_world_bringup/meshes/rlink2.STL; visual mesh filename=package://m3pro_world_bringup/meshes/rlink2.STL
- link rlink3: geometry collision mesh filename=package://m3pro_world_bringup/meshes/rlink3.STL; visual mesh filename=package://m3pro_world_bringup/meshes/rlink3.STL
- link rwheel1: geometry collision cylinder length=0.02 radius=0.04; visual mesh filename=package://m3pro_world_bringup/meshes/rwheel1.STL
- link rwheel2: geometry collision cylinder length=0.02 radius=0.04; visual mesh filename=package://m3pro_world_bringup/meshes/rwheel2.STL
Joints:
- removed joint laser_front_right_joint_to_remove
- removed joint laser_rear_left_joint_to_remove
