Commit message: Suspended-obstacle avoidance

File: src/m3pro_world_bringup/urdf/M3Pro.urdf (robot description, URDF)
Before this commit: robot M3Pro, 25 links, 24 joints
Joints:
- joint arm2_Joint: origin xyz=-0.0021522 6.1185E-05 0.033 rpy=0 -${pi/4} 0 -> xyz=-0.0021522 6.1185E-05 0.033 rpy=0 -0.7854 0
- joint arm3_Joint: origin xyz=0 0 0.08285 rpy=0 ${pi/2} 0 -> xyz=0 0 0.08285 rpy=0 1.5708 0
- joint arm4_Joint: origin xyz=0 0 0.08285 rpy=0 ${pi/4} 0 -> xyz=0 0 0.08285 rpy=0 0.7854 0
- joint camera_optical_joint: origin xyz=0 0 0 rpy=${-pi/2} 0 ${-pi/2} -> xyz=0 0 0 rpy=-1.5708 0 -1.5708
- joint laser_rear_joint: origin xyz=-0.11867 0.09 0.1253 rpy=0 0 ${pi} -> xyz=-0.11867 0.09 0.1253 rpy=0 0 3.1416
